File: PCBs/Charger/Charger.sch (KiCad schematic (older format))
At the start: 18 parts, among them J1 Battery, J2 Charger, J3 Output 1, J4 Output 2, J5 MCU, U1 MCP73831T-2, U2 MAX17048

Commit message: New circuits
Parts:
- R1: value 1K -> 2K
Changed lines of the file:
@@
 P 5200 4350
 F 0 "R1" H 5268 4396 50  0000 L CNN
-F 1 "1K" H 5268 4305 50  0000 L CNN
+F 1 "2K" H 5268 4305 50  0000 L CNN
 F 2 "Resistors_SMD:R_0805_HandSoldering" V 5240 4340 50  0001 C CNN
 F 3 "~" H 5200 4350 50  0001 C CNN

Commit message: Changed
Parts:
- removed C4: 10nF, Resistors_SMD:R_0805_HandSoldering, symbol Device:C
- removed J4: Output 2, Pin_Headers:Pin_Header_Straight_1x02_Pitch2.54mm, symbol Connector_Generic:Conn_01x02
- removed J5: MCU, Pin_Headers:Pin_Header_Straight_1x08_Pitch2.54mm, symbol Connector_Generic:Conn_01x08
- removed R2: 1K, Resistors_SMD:R_0805_HandSoldering, symbol Device:R_US
- added C3: 10uF, Resistors_SMD:R_0805_HandSoldering, symbol Device:C
- added J4: MCU, Pin_Headers:Pin_Header_Angled_1x09_Pitch2.54mm, symbol Connector_Generic:Conn_01x09
- added L1: 1uH, Inductors_SMD:L_0805_HandSoldering, symbol pspice:INDUCTOR
- added R5: 1K, Resistors_SMD:R_0805_HandSoldering, symbol Device:R_US
- added U2: TPS61240, my-smd:WSON6_2.1x2.1mm_Pitch0.65mm, symbol my-regulators:TPS61240
- J3: value Output 1 -> LEDs
- R3: renamed from R7; value 4.7K -> 2.2K
- R4: value 150 -> 3.3K
- U1: footprint TO_SOT_Packages_SMD:SOT-23-5_HandSoldering -> my-smd:SOT-23-5_HandSoldering
- renumbered C3 to C4, R3 to R1, R1 to R2, R5 to R6, R6 to R7, U2 to U3
Connections:
- net 3.3V: now also J4.3 (Pin_3); no longer R4.1
- net GND: now also R4.2, U3.6 (QSTRT), C3.2, J4.1 (Pin_1), U2.1 (GND); no longer R3.2
- net SCL: now also J4.6 (Pin_6)
- net SDA: now also J4.9 (Pin_9)
- net VBAT: now also J4.2 (Pin_2), L1.1, R5.1, U2.6 (VIN); no longer J3.1 (Pin_1)
- net VCHG: now also R3.1
- net STAT: now reaches R1.2, U1.1 (STAT)
- net ~CHG_EN: now reaches R2.1, U1.5 (PROG)
- net ~CHG_EN: now also J4.7 (Pin_7)
- net CELL: now reaches C4.1, U3.2 (CELL)
- net CELL: now also U3.3 (VDD), R5.2
- removed net QSTRT: R3.1, U3.6 (QSTRT)
- net ~ALRT: no longer names the net of U3.5 (~ALRT)
- net ~STAT renamed ~CHARGING
- net ~CHARGING: now also J4.4 (Pin_4)
- new net CHG_PRESENT: J4.5 (Pin_5), R3.2, R4.1
- new net L: L1.2, U2.5 (L)
- new net LED_EN: J4.8 (Pin_8), U2.4 (EN)
- new net VLED: C3.1, J3.1 (Pin_1), U2.2 (VOUT), U2.3 (FB)
- no-connect marks 0 -> 1
Other:
- moved on the sheet: C1, C2, C4, J1, J2, J3, R1, R2, R3, R6, R7, U1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

Commit message: Fixed some output pins.
Parts:
- added R5: 4.7K, Resistors_SMD:R_0805_HandSoldering, symbol Device:R_US
- U2: symbol my-regulators:TPS61240 -> Charger-rescue:TPS61240-my-regulators
- U3: symbol maxim:MAX17043 -> Charger-rescue:MAX17043-maxim
- renumbered R5 to R6, R6 to R7, R7 to R8
Connections:
- net GND: now also R5.2
- net LED_EN: now also J4.9 (Pin_9), R5.1; no longer J4.8 (Pin_8)
- net SDA: now also J4.7 (Pin_7); no longer J4.9 (Pin_9)
- net ~CHG_EN: now also J4.8 (Pin_8); no longer J4.7 (Pin_7)
Changed lines of the file:
@@
 $EndDescr
 $Comp
-L maxim:MAX17043 U3
+L Charger-rescue:MAX17043-maxim U3
 U 1 1 5DB70484
 P 7250 3150
@@
 Text Label 8150 1800 0    50   ~ 0
 VBAT
-Text Label 8200 3800 0    50   ~ 0
+Text Label 8150 3600 0    50   ~ 0
 SDA
 Text Label 8450 3500 0    50   ~ 0
@@
 Connection ~ 2000 4950
 $Comp
-L Device:R_US R6
+L Device:R_US R7
 U 1 1 5DB9E613
 P 8000 3050
-F 0 "R6" H 8068 3096 50  0000 L CNN
+F 0 "R7" H 8068 3096 50  0000 L CNN
 F 1 "4.7K" H 8068 3005 50  0000 L CNN
 F 2 "Resistors_SMD:R_0805_HandSoldering" V 8040 3040 50  0001 C CNN
@@
 $EndComp
 $Comp
-L Device:R_US R7
+L Device:R_US R8
 U 1 1 5DBA021B
 P 8300 3050
-F 0 "R7" H 8368 3096 50  0000 L CNN
+F 0 "R8" H 8368 3096 50  0000 L CNN
 F 1 "4.7K" H 8368 3005 50  0000 L CNN
 F 2 "Resistors_SMD:R_0805_HandSoldering" V 8340 3040 50  0001 C CNN
@@
 	2450 1800 2450 3500
 $Comp
-L Device:R_US R5
+L Device:R_US R6
 U 1 1 5DC6C6A1
 P 6500 2650
-F 0 "R5" H 6568 2696 50  0000 L CNN
+F 0 "R6" H 6568 2696 50  0000 L CNN
 F 1 "1K" H 6568 2605 50  0000 L CNN
 F 2 "Resistors_SMD:R_0805_HandSoldering" V 6540 2640 50  0001 C CNN
@@
 	6750 2550 7300 2550
 $Comp
-L my-regulators:TPS61240 U2
+L Charger-rescue:TPS61240-my-regulators U2
 U 1 1 5DC514F8
 P 5100 3550
@@
 Connection ~ 4200 4950
 Wire Wire Line
-	4200 4950 5700 4950
+	4200 4950 4550 4950
 Wire Wire Line
 	4200 4550 4200 4350
@@
 	4400 1800 6500 1800
 Wire Wire Line
-	8000 3300 8000 3800
-Wire Wire Line
-	8000 3800 9000 3800
+	8000 3300 8000 3600
 Connection ~ 8000 3300
 Wire Wire Line
@@
 	8300 3500 9000 3500
 Connection ~ 8300 3400
-Wire Wire Line
-	8450 4150 8450 3700
-Wire Wire Line
-	8450 3700 9000 3700
-Wire Wire Line
-	8550 4250 8550 3600
-Wire Wire Line
-	8550 3600 9000 3600
 Wire Wire Line
 	8650 4350 8650 3400
@@
 Text Label 6500 3100 0    50   ~ 0
 CELL
+Wire Wire Line
+	8000 3600 9000 3600
+Wire Wire Line
+	8550 4250 8550 3700
+Wire Wire Line
+	8550 3700 9000 3700
+Wire Wire Line
+	8450 4150 8450 3800
+Wire Wire Line
+	8450 3800 9000 3800
+$Comp
+L Device:R_US R5
+U 1 1 5DC1CF62
+P 4550 4700
+F 0 "R5" H 4618 4746 50  0000 L CNN
+F 1 "4.7K" H 4618 4655 50  0000 L CNN
+F 2 "Resistors_SMD:R_0805_HandSoldering" V 4590 4690 50  0001 C CNN
+F 3 "~" H 4550 4700 50  0001 C CNN
+	1    4550 4700
+	1    0    0    -1
+$EndComp
+Wire Wire Line
+	4550 4550 4550 4150
+Connection ~ 4550 4150
+Wire Wire Line
+	4550 4850 4550 4950
+Connection ~ 4550 4950
+Wire Wire Line
+	4550 4950 5700 4950
 $EndSCHEMATC

Commit message: New design and layout
Parts:
- removed J4: MCU, Pin_Headers:Pin_Header_Angled_1x09_Pitch2.54mm, symbol Connector_Generic:Conn_01x09
- removed R7, R8: 4.7K, Resistors_SMD:R_0805_HandSoldering, symbol Device:R_US
- added J4: MCU, Pin_Headers:Pin_Header_Straight_1x08_Pitch2.54mm, symbol Connector_Generic:Conn_01x08
- R5: value 4.7K -> 10K
Connections:
- net CHG_PRESENT: now also J4.4 (Pin_4)
- net GND: now also J4.1 (Pin_1)
- net LED_EN: now also J4.8 (Pin_8)
- net SCL: now also J4.5 (Pin_5)
- net SDA: now also J4.6 (Pin_6)
- net VBAT: now also J4.2 (Pin_2)
- net ~CHARGING: now also J4.3 (Pin_3)
- net ~CHG_EN: now also J4.7 (Pin_7)
Other:
- moved on the sheet: L1
Changed lines of the file:
@@
 Connection ~ 3900 4950
-Wire Wire Line
-	8550 3200 9000 3200
 Wire Wire Line
 	6650 3400 6650 3800
@@
 	9000 2300 8900 2300
 Connection ~ 6750 2900
-Text Label 8450 2800 0    50   ~ 0
-3.3V
 Text Label 8150 1800 0    50   ~ 0
 VBAT
-Text Label 8150 3600 0    50   ~ 0
+Text Label 8150 3500 0    50   ~ 0
 SDA
-Text Label 8450 3500 0    50   ~ 0
+Text Label 8150 3400 0    50   ~ 0
 SCL
 Text Label 8100 4950 0    50   ~ 0
@@
 Connection ~ 2000 4950
 $Comp
-L Device:R_US R7
-U 1 1 5DB9E613
-P 8000 3050
-F 0 "R7" H 8068 3096 50  0000 L CNN
-F 1 "4.7K" H 8068 3005 50  0000 L CNN
-F 2 "Resistors_SMD:R_0805_HandSoldering" V 8040 3040 50  0001 C CNN
-F 3 "~" H 8000 3050 50  0001 C CNN
-	1    8000 3050
-	1    0    0    -1
-$EndComp
-$Comp
-L Device:R_US R8
-U 1 1 5DBA021B
-P 8300 3050
-F 0 "R8" H 8368 3096 50  0000 L CNN
-F 1 "4.7K" H 8368 3005 50  0000 L CNN
-F 2 "Resistors_SMD:R_0805_HandSoldering" V 8340 3040 50  0001 C CNN
-F 3 "~" H 8300 3050 50  0001 C CNN
-	1    8300 3050
-	1    0    0    -1
-$EndComp
-Wire Wire Line
-	8000 2800 8000 2900
-Wire Wire Line
-	8000 2800 8300 2800
-Wire Wire Line
-	8300 2800 8300 2900
-Wire Wire Line
-	8550 2800 8550 3200
-Connection ~ 8300 2800
-$Comp
 L Device:R_US R3
 U 1 1 5DBA57A4
@@
 	7750 2900 7850 2900
 Wire Wire Line
-	8300 2800 8550 2800
-Wire Wire Line
 	8750 3100 9000 3100
 Wire Wire Line
 	8900 3000 9000 3000
-Wire Wire Line
-	8000 3300 8000 3200
 Wire Wire Line
 	7850 2550 7850 2900
@@
 L pspice:INDUCTOR L1
 U 1 1 5DCCC5EF
-P 4750 2900
-F 0 "L1" H 4750 3115 50  0000 C CNN
-F 1 "1uH" H 4750 3024 50  0000 C CNN
-F 2 "Inductors_SMD:L_0805_HandSoldering" H 4750 2900 50  0001 C CNN
-F 3 "~" H 4750 2900 50  0001 C CNN
-	1    4750 2900
-	1    0    0    -1
+P 4550 2600
+F 0 "L1" V 4450 2700 50  0000 C CNN
+F 1 "1uH" V 4550 2724 50  0000 C CNN
+F 2 "Inductors_SMD:L_0805_HandSoldering" H 4550 2600 50  0001 C CNN
+F 3 "~" H 4550 2600 50  0001 C CNN
+	1    4550 2600
+	0    1    1    0
 $EndComp
 Wire Wire Line
 	4650 3450 4400 3450
-Wire Wire Line
-	4400 3450 4400 2900
 Connection ~ 4400 1800
-Wire Wire Line
-	4500 2900 4400 2900
-Connection ~ 4400 2900
-Wire Wire Line
-	4400 2900 4400 1800
-Wire Wire Line
-	5000 2900 5100 2900
-Wire Wire Line
-	5100 2900 5100 3050
-Wire Wire Line
-	5100 3050 4550 3050
-Wire Wire Line
-	4550 3050 4550 3550
 Wire Wire Line
 	4550 3550 4650 3550
@@
 	8750 1800 6500 1800
 Connection ~ 6500 1800
-$Comp
-L Connector_Generic:Conn_01x09 J4
-U 1 1 5DD0A71E
-P 9200 3400
-F 0 "J4" H 9279 3442 50  0000 L CNN
-F 1 "MCU" H 9279 3351 50  0000 L CNN
-F 2 "Pin_Headers:Pin_Header_Angled_1x09_Pitch2.54mm" H 9200 3400 50  0001 C CNN
-F 3 "~" H 9200 3400 50  0001 C CNN
-	1    9200 3400
-	1    0    0    -1
-$EndComp
 Wire Wire Line
 	8450 4150 4550 4150
@@
 	5950 2200 9000 2200
 Wire Wire Line
-	7750 3400 8300 3400
-Wire Wire Line
-	8300 3200 8300 3400
-Wire Wire Line
 	4400 1800 6500 1800
 Wire Wire Line
-	8000 3300 8000 3600
-Connection ~ 8000 3300
-Wire Wire Line
-	8300 3400 8300 3500
-Wire Wire Line
-	8300 3500 9000 3500
-Connection ~ 8300 3400
-Wire Wire Line
-	8650 4350 8650 3400
-Wire Wire Line
-	8650 3400 9000 3400
-Wire Wire Line
-	8750 4450 8750 3300
-Wire Wire Line
-	8750 3300 9000 3300
+	8000 3300 8000 3500
 Text Label 6750 2200 0    50   ~ 0
 VLED
 Text Label 2900 4050 0    50   ~ 0
 STAT
-Text Label 4650 3050 0    50   ~ 0
+Text Label 4550 3050 0    50   ~ 0
 L
 Text Label 6500 3100 0    50   ~ 0
 CELL
-Wire Wire Line
-	8000 3600 9000 3600
-Wire Wire Line
-	8550 4250 8550 3700
-Wire Wire Line
-	8550 3700 9000 3700
-Wire Wire Line
-	8450 4150 8450 3800
-Wire Wire Line
-	8450 3800 9000 3800
 $Comp
 L Device:R_US R5
@@
 P 4550 4700
 F 0 "R5" H 4618 4746 50  0000 L CNN
-F 1 "4.7K" H 4618 4655 50  0000 L CNN
+F 1 "10K" H 4618 4655 50  0000 L CNN
 F 2 "Resistors_SMD:R_0805_HandSoldering" V 4590 4690 50  0001 C CNN
 F 3 "~" H 4550 4700 50  0001 C CNN
@@
 Wire Wire Line
 	4550 4950 5700 4950
+Wire Wire Line
+	8750 3200 9000 3200
+Wire Wire Line
+	8750 3200 8750 4450
+Wire Wire Line
+	8650 3300 9000 3300
+Wire Wire Line
+	8650 3300 8650 4350
+Wire Wire Line
+	7750 3400 9000 3400
+Wire Wire Line
+	9000 3500 8000 3500
+Wire Wire Line
+	8550 3600 9000 3600
+Wire Wire Line
+	8550 3600 8550 4250
+Wire Wire Line
+	8450 3700 9000 3700
+Wire Wire Line
+	8450 3700 8450 4150
+$Comp
+L Connector_Generic:Conn_01x08 J4
+U 1 1 5DC3011D
+P 9200 3300
+F 0 "J4" H 9279 3292 50  0000 L CNN
+F 1 "MCU" H 9279 3201 50  0000 L CNN
+F 2 "Pin_Headers:Pin_Header_Straight_1x08_Pitch2.54mm" H 9200 3300 50  0001 C CNN
+F 3 "~" H 9200 3300 50  0001 C CNN
+	1    9200 3300
+	1    0    0    -1
+$EndComp
+Wire Wire Line
+	4400 1800 4400 2200
+Wire Wire Line
+	4400 2200 4550 2200
+Wire Wire Line
+	4550 2200 4550 2350
+Connection ~ 4400 2200
+Wire Wire Line
+	4400 2200 4400 3450
+Wire Wire Line
+	4550 2850 4550 3550
 $EndSCHEMATC
