File: PCBs/Connector/Connector.kicad_pcb (KiCad board)
At the start: 2 copper layers, 6.7 x 83 mm, 3 parts, among them J1 MCU, J2 Accel, J3 Charger

Commit message: Started firmware
Other:
- board text added: "Connector v1"
Changed lines of the file:
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@@
   (general
     (thickness 1.6)
-    (drawings 11)
+    (drawings 12)
     (tracks 52)
     (zones 0)
@@
   )
   (page A4)
+  (title_block
+    (title "Connector v1")
+  )
   (layers
     (0 F.Cu signal)
@@
     )
   )
+  (gr_text "Connector v1" (at 137.7 70.8 90) (layer F.SilkS)
+    (effects (font (size 1.5 1.5) (thickness 0.3)))
+  )
   (gr_line (start 135.4 137.2) (end 139.5 133.1) (layer Edge.Cuts) (width 0.15))

Commit message: New designs
Parts:
- J1: footprint Pin_Headers:Pin_Header_Straight_1x13_Pitch2.54mm -> Pin_Headers:Pin_Header_Straight_1x15_Pitch2.54mm
- J3: value Charger -> Power Supply
- moved J2 31.5 mm to (165.1, 99.1)
- moved J3 31.3 mm to (165.1, 121.9)
- moved J1 31.1 mm to (165.1, 55.9)
Connections:
- net /~ALRT renamed /~CHG_EN
- net /~STAT renamed /LED_EN
- J1 pad 10: (no net) -> /AC_INT2
- J1 pad 11: /3.3V -> (no net)
- J1 pad 12: /VBAT -> (no net)
- J1 pad 13: /GND -> /3.3V
- J1 pad 3: /QSTRT -> /SDA
- J1 pad 4: /AC_CS -> (no net)
- J1 pad 5: /AC_INT1 -> (no net)
- J1 pad 6: /AC_INT2 -> /SCL
- J1 pad 7: /SDA -> /CHG_PRESENT
- J1 pad 8: /SCL -> /~CHARGING
- J1 pad 9: (no net) -> /AC_INT1
- J2 pad 3: (no net) -> /3.3V
- J2 pad 6: /AC_CS -> /3.3V
- J3 pad 3: /3.3V -> /~CHARGING
- J3 pad 4: /SDA -> /CHG_PRESENT
- J3 pad 6: /QSTRT -> /SDA
Routing:
- net /QSTRT: track 73.9 -> 0.00 mm
- net /CHG_PRESENT: track 0.00 -> 63.3 mm, vias 0 -> 2
- net /~CHARGING: track 0.00 -> 59.3 mm
- net /AC_CS: track 47.2 -> 0.00 mm
- net /GND: track 34.1 -> 0.00 mm, vias 0 -> 10
- net /SDA: track 74.3 -> 102.8 mm
- net /3.3V: track 57.4 -> 34.7 mm, vias 1 -> 2
- net /SCL: track 79.0 -> 91.5 mm, vias 1 -> 2
- net /AC_INT2: track 36.2 -> 31.1 mm, vias 0 -> 1
- net /AC_INT1: track 41.7 -> 36.7 mm, vias 0 -> 1
- net /~CHG_EN: track 79.4 -> 84.2 mm
- net /LED_EN: track 84.5 -> 89.2 mm
- net /VBAT: track 39.2 -> 37.4 mm
- added copper zone on B.Cu, net /GND
- added copper zone on F.Cu, net /GND
Other:
- board size 6.7 x 83 mm -> 9.1 x 86.4 mm
