File: PCBs/IRBlasterFP/IRBlasterFP.kicad_pcb (KiCad board)
At the start: 2 copper layers, 0 parts

Commit message: New designs
Parts:
- added C1: 1uF, Capacitors_THT:CP_Radial_D5.0mm_P2.50mm, F.Cu at (159.0, 95.4)
- added D1: IR_OUT, LEDs:LED_D3.0mm, F.Cu at (141.0, 94.0)
- added D2: STATUS, LEDs:LED_D3.0mm, F.Cu at (153.7, 94.0)
- added J1: Front Panel, Pin_Headers:Pin_Header_Straight_1x05_Pitch2.54mm, F.Cu at (157.5, 100.3)
- added R1: 750, Resistors_THT:R_Axial_DIN0204_L3.6mm_D1.6mm_P1.90mm_Vertical, F.Cu at (144.5, 97.0)
- added R2: 750, Resistors_THT:R_Axial_DIN0204_L3.6mm_D1.6mm_P1.90mm_Vertical, F.Cu at (147.6, 97.0)
- added REF**: MountingHole_3.2mm_M3, Mounting_Holes:MountingHole_3.2mm_M3, F.Cu at (165.1, 100.3)
- added REF**: MountingHole_3.2mm_M3, Mounting_Holes:MountingHole_3.2mm_M3, F.Cu at (139.7, 100.3)
- added U1: TSOP38238, Pin_Headers:Pin_Header_Straight_1x03_Pitch2.54mm, F.Cu at (167.6, 94.0)
Routing:
- net /IR_IN: track 0.00 -> 19.9 mm
- net /3.3V: track 0.00 -> 9.72 mm
- net Net-(D1-Pad2): track 0.00 -> 7.09 mm
- net /IR_OUT: track 0.00 -> 4.46 mm
- net /STATUS: track 0.00 -> 4.25 mm
- net Net-(D2-Pad2): track 0.00 -> 4.03 mm
- added copper zone on B.Cu, net /GND
- added copper zone on F.Cu, net /GND
Other:
- board outline added: 33 x 12.7 mm
- board text added: "IRBlasterFP v1"

Commit message: Fixed problems
Other:
- rule pad_to_mask_clearance: 0.2 -> 0.0508
- board text added: "IRBlasterFP v2"
- board text removed: "IRBlasterFP v1"
Changed lines of the file:
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@@
   )
   (page A4)
+  (title_block
+    (title "IRBlaster FP v2")
+  )
   (layers
     (0 F.Cu signal)
@@
     (last_trace_width 0.1524)
     (trace_clearance 0.1524)
-    (zone_clearance 0.508)
+    (zone_clearance 0.3048)
     (zone_45_only no)
     (trace_min 0.1524)
@@
     (pad_size 1.524 1.524)
     (pad_drill 0.762)
-    (pad_to_mask_clearance 0.2)
+    (pad_to_mask_clearance 0.0508)
     (solder_mask_min_width 0.25)
     (aux_axis_origin 0 0)
@@
     (pad 1 np_thru_hole circle (at 0 0) (size 3.2 3.2) (drill 3.2) (layers *.Cu *.Mask))
   )
-  (gr_text "IRBlasterFP v1\n" (at 152.4 102.87) (layer F.SilkS)
+  (gr_text "IRBlasterFP v2\n" (at 152.4 102.87) (layer F.SilkS)
     (effects (font (size 1.2 1.2) (thickness 0.2)))
   )
@@
   (segment (start 147.574 95.128) (end 149.982 95.128) (width 0.1524) (layer F.Cu) (net 7))
   (zone (net 1) (net_name /GND) (layer F.Cu) (hatch edge 0.508)
-    (connect_pads yes (clearance 0.1524))
+    (connect_pads yes (clearance 0.3048))
     (min_thickness 0.1524)
     (fill yes (arc_segments 16) (thermal_gap 0.508) (thermal_bridge_width 0.508))
@@
   )
   (zone (net 1) (net_name /GND) (layer B.Cu) (hatch edge 0.508)
-    (connect_pads yes (clearance 0.1524))
+    (connect_pads yes (clearance 0.3048))
     (min_thickness 0.1524)
     (fill yes (arc_segments 16) (thermal_gap 0.508) (thermal_bridge_width 0.508))
