File: PCBs/IRBlaster/IRBlaster.sch (KiCad schematic (older format))
At the start: 21 parts, among them J1 Raspberry Pi, J2 Power, J3 Regulator, J4 Front Panel 1, J5 Blaster 1, J6 Blaster 2, J7 Blaster 3, J8 Blaster 4, Q1 ZTX602/3, Q2 ZTX602/3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

Commit message: Changed
Parts:
- removed C1: 10uF, Capacitors_THT:CP_Radial_D5.0mm_P2.50mm, symbol Device:CP1
- removed J1: Raspberry Pi, Pin_Headers:Pin_Header_Straight_2x04_Pitch2.54mm, symbol Connector_Generic:Conn_02x04_Top_Bottom
- removed Q1, Q2, Q3, Q4: ZTX602/3, my-transistors:TO-92_Inline_Wide_Reverse, symbol Device:Q_NPN_Darlington_CBE
- added C1: 10uF, Capacitor_SMD:C_0805_2012Metric_Pad1.15x1.40mm_HandSolder, symbol Device:C
- added J1: Raspberry Pi, Connector_PinHeader_2.54mm:PinHeader_2x04_P2.54mm_Vertical, symbol Connector_Generic:Conn_02x04_Odd_Even
- added Q1, Q2, Q3, Q4: IRLML6244, Package_TO_SOT_SMD:SOT-23_Handsoldering, symbol Transistor_FET:2N7002
- J2: footprint terminals:Terminal_5mm_2pos -> Connector_PinHeader_2.54mm:PinHeader_1x02_P2.54mm_Vertical
- J5, J6, J7, J8: footprint Pin_Headers:Pin_Header_Straight_1x02_Pitch2.54mm -> Connector_PinHeader_2.54mm:PinHeader_1x02_P2.54mm_Vertical
- R1, R2, R3, R5, R6, R7, R8: footprint Resistors_THT:R_Axial_DIN0204_L3.6mm_D1.6mm_P2.54mm_Vertical -> Resistor_SMD:R_0805_2012Metric_Pad1.15x1.40mm_HandSolder
- R4: value 4K -> 100; footprint Resistors_THT:R_Axial_DIN0204_L3.6mm_D1.6mm_P2.54mm_Vertical -> Resistor_SMD:R_0805_2012Metric_Pad1.15x1.40mm_HandSolder
Connections:
- net 3.3V: now also J1.1 (Pin_1)
- net 5V: now also C1.1, J1.2 (Pin_2), J1.4 (Pin_4)
- net GND: now also C1.2, J1.6 (Pin_6), Q1.2 (S), Q2.2 (S), Q3.2 (S), Q4.2 (S)
- net IR_IN: now also J4.3 (Pin_3), J1.3 (Pin_3); no longer J4.5 (Pin_5)
- net IR_OUT: now also J1.7 (Pin_7)
- net STATUS: now also J1.5 (Pin_5)
- net at R3.2: now also J4.5 (Pin_5); no longer J4.3 (Pin_3)
- net IRB_1: now reaches J5.2 (Pin_2), R5.1
- net IRB_2: now reaches J6.2 (Pin_2), R6.1
- net IRB_3: now reaches J7.2 (Pin_2), R7.1
- net IRB_4: now reaches J8.2 (Pin_2), R8.1
- net at R5.2: now also Q1.3 (D)
- net at R4.1: now also Q1.1 (G), Q2.1 (G), Q3.1 (G), Q4.1 (G)
- net at R6.2: now also Q2.3 (D)
- net at R7.2: now also Q3.3 (D)
- net at R8.2: now also Q4.3 (D)

Commit message: New designs
Parts:
- removed R1, R3: 750, Resistor_SMD:R_0805_2012Metric_Pad1.15x1.40mm_HandSolder, symbol Device:R_US
- J4: value Front Panel 1 -> Front Panel
- renumbered R2 to R1, R4 to R2, R5 to R3, R6 to R4, R7 to R5, R8 to R6
Connections:
- net IR_OUT: now also J4.5 (Pin_5)
- net STATUS: now also J4.4 (Pin_4)
Changed lines of the file:
@@
 P 2200 4100
 F 0 "J4" H 2120 4517 50  0000 C CNN
-F 1 "Front Panel 1" H 2120 4426 50  0000 C CNN
+F 1 "Front Panel" H 2120 4426 50  0000 C CNN
 F 2 "Pin_Headers:Pin_Header_Straight_1x05_Pitch2.54mm" H 2200 4100 50  0001 C CNN
 F 3 "~" H 2200 4100 50  0001 C CNN
@@
 $EndComp
 $Comp
-L Device:R_US R2
+L Device:R_US R1
 U 1 1 5DBC6D56
 P 3200 3450
-F 0 "R2" H 3268 3496 50  0000 L CNN
+F 0 "R1" H 3268 3496 50  0000 L CNN
 F 1 "10K" H 3268 3405 50  0000 L CNN
 F 2 "Resistor_SMD:R_0805_2012Metric_Pad1.15x1.40mm_HandSolder" V 3240 3440 50  0001 C CNN
@@
 $EndComp
 $Comp
-L Device:R_US R1
-U 1 1 5DBC75E9
-P 2800 3450
-F 0 "R1" H 2868 3496 50  0000 L CNN
-F 1 "750" H 2868 3405 50  0000 L CNN
-F 2 "Resistor_SMD:R_0805_2012Metric_Pad1.15x1.40mm_HandSolder" V 2840 3440 50  0001 C CNN
-F 3 "~" H 2800 3450 50  0001 C CNN
-	1    2800 3450
-	1    0    0    -1
-$EndComp
-$Comp
 L Device:R_US R3
-U 1 1 5DBC7689
-P 3600 3450
-F 0 "R3" H 3668 3496 50  0000 L CNN
-F 1 "750" H 3668 3405 50  0000 L CNN
-F 2 "Resistor_SMD:R_0805_2012Metric_Pad1.15x1.40mm_HandSolder" V 3640 3440 50  0001 C CNN
-F 3 "~" H 3600 3450 50  0001 C CNN
-	1    3600 3450
-	1    0    0    -1
-$EndComp
-$Comp
-L Device:R_US R5
 U 1 1 5DBC78D7
 P 4700 2650
-F 0 "R5" H 4768 2696 50  0000 L CNN
+F 0 "R3" H 4768 2696 50  0000 L CNN
 F 1 "0" H 4768 2605 50  0000 L CNN
 F 2 "Resistor_SMD:R_0805_2012Metric_Pad1.15x1.40mm_HandSolder" V 4740 2640 50  0001 C CNN
@@
 $EndComp
 $Comp
-L Device:R_US R4
+L Device:R_US R2
 U 1 1 5DBC793D
 P 3950 3100
-F 0 "R4" V 3745 3100 50  0000 C CNN
+F 0 "R2" V 3745 3100 50  0000 C CNN
 F 1 "100" V 3836 3100 50  0000 C CNN
 F 2 "Resistor_SMD:R_0805_2012Metric_Pad1.15x1.40mm_HandSolder" V 3990 3090 50  0001 C CNN
@@
 $EndComp
 $Comp
-L Device:R_US R6
+L Device:R_US R4
 U 1 1 5DBC8AAB
 P 4700 3850
-F 0 "R6" H 4768 3896 50  0000 L CNN
+F 0 "R4" H 4768 3896 50  0000 L CNN
 F 1 "0" H 4768 3805 50  0000 L CNN
 F 2 "Resistor_SMD:R_0805_2012Metric_Pad1.15x1.40mm_HandSolder" V 4740 3840 50  0001 C CNN
@@
 	3200 3100 3200 3300
 Connection ~ 3200 3100
-Wire Wire Line
-	3600 3300 3600 3100
 Connection ~ 3600 3100
 Wire Wire Line
@@
 Text Label 4050 1100 0    50   ~ 0
 IR_IN
-Wire Wire Line
-	2800 4200 2800 3600
-Wire Wire Line
-	2800 3300 2800 1200
 $Comp
 L Transistor_FET:2N7002 Q1
@@
 	3050 1100 4700 1100
 Wire Wire Line
-	3600 3600 3600 4300
-Wire Wire Line
 	2400 4300 3600 4300
 Wire Wire Line
@@
 $EndComp
 $Comp
-L Device:R_US R7
+L Device:R_US R5
 U 1 1 5DBDB627
 P 4700 5050
-F 0 "R7" H 4768 5096 50  0000 L CNN
+F 0 "R5" H 4768 5096 50  0000 L CNN
 F 1 "0" H 4768 5005 50  0000 L CNN
 F 2 "Resistor_SMD:R_0805_2012Metric_Pad1.15x1.40mm_HandSolder" V 4740 5040 50  0001 C CNN
@@
 Connection ~ 5800 3500
 $Comp
-L Device:R_US R8
+L Device:R_US R6
 U 1 1 5DBDF64E
 P 4700 6250
-F 0 "R8" H 4768 6296 50  0000 L CNN
+F 0 "R6" H 4768 6296 50  0000 L CNN
 F 1 "0" H 4768 6205 50  0000 L CNN
 F 2 "Resistor_SMD:R_0805_2012Metric_Pad1.15x1.40mm_HandSolder" V 4740 6240 50  0001 C CNN
@@
 Text Label 5150 6000 0    50   ~ 0
 IRB_4
+Wire Wire Line
+	3600 3100 3600 4300
+Wire Wire Line
+	2800 1200 2800 4200
 $EndSCHEMATC

Commit message: Set emitter resistor values
Parts:
- R3, R4, R5, R6: value 0 -> 1K
Changed lines of the file:
@@
 P 4700 2650
 F 0 "R3" H 4768 2696 50  0000 L CNN
-F 1 "0" H 4768 2605 50  0000 L CNN
+F 1 "1K" H 4768 2605 50  0000 L CNN
 F 2 "Resistor_SMD:R_0805_2012Metric_Pad1.15x1.40mm_HandSolder" V 4740 2640 50  0001 C CNN
 F 3 "~" H 4700 2650 50  0001 C CNN
@@
 P 4700 3850
 F 0 "R4" H 4768 3896 50  0000 L CNN
-F 1 "0" H 4768 3805 50  0000 L CNN
+F 1 "1K" H 4768 3805 50  0000 L CNN
 F 2 "Resistor_SMD:R_0805_2012Metric_Pad1.15x1.40mm_HandSolder" V 4740 3840 50  0001 C CNN
 F 3 "~" H 4700 3850 50  0001 C CNN
@@
 P 4700 5050
 F 0 "R5" H 4768 5096 50  0000 L CNN
-F 1 "0" H 4768 5005 50  0000 L CNN
+F 1 "1K" H 4768 5005 50  0000 L CNN
 F 2 "Resistor_SMD:R_0805_2012Metric_Pad1.15x1.40mm_HandSolder" V 4740 5040 50  0001 C CNN
 F 3 "~" H 4700 5050 50  0001 C CNN
@@
 P 4700 6250
 F 0 "R6" H 4768 6296 50  0000 L CNN
-F 1 "0" H 4768 6205 50  0000 L CNN
+F 1 "1K" H 4768 6205 50  0000 L CNN
 F 2 "Resistor_SMD:R_0805_2012Metric_Pad1.15x1.40mm_HandSolder" V 4740 6240 50  0001 C CNN
 F 3 "~" H 4700 6250 50  0001 C CNN
