File: PCBs/IRBlaster/IRBlaster.kicad_pcb (KiCad board)
At the start: 2 copper layers, 28 x 48.3 mm, 21 parts, among them J1 Raspberry Pi, J2 Power, J3 Regulator, J4 Front Panel 1, J5 Blaster 1, J6 Blaster 2, J7 Blaster 3, J8 Blaster 4, Q1 ZTX602/3, Q2 ZTX602/3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

Commit message: Changed
Parts:
- added REF**: Brace, Connector_PinHeader_2.54mm:PinHeader_1x02_P2.54mm_Vertical, F.Cu at (190.5, 111.8)
- C1: footprint Capacitors_THT:CP_Radial_D5.0mm_P2.50mm -> Capacitor_SMD:C_0805_2012Metric_Pad1.15x1.40mm_HandSolder
- J1: footprint Pin_Headers:Pin_Header_Straight_2x04_Pitch2.54mm -> Connector_PinHeader_2.54mm:PinHeader_2x04_P2.54mm_Vertical
- J2: footprint terminals:Terminal_5mm_2pos -> Connector_PinHeader_2.54mm:PinHeader_1x02_P2.54mm_Vertical
- J5, J6, J7, J8: footprint Pin_Headers:Pin_Header_Straight_1x02_Pitch2.54mm -> Connector_PinHeader_2.54mm:PinHeader_1x02_P2.54mm_Vertical
- Q1, Q2, Q3, Q4: value ZTX602/3 -> IRLML6244; footprint my-transistors:TO-92_Inline_Wide_Reverse -> Package_TO_SOT_SMD:SOT-23_Handsoldering
- R1, R2, R3, R5, R6, R7, R8: footprint Resistors_THT:R_Axial_DIN0204_L3.6mm_D1.6mm_P2.54mm_Vertical -> Resistor_SMD:R_0805_2012Metric_Pad1.15x1.40mm_HandSolder
- R4: value 4K -> 100; footprint Resistors_THT:R_Axial_DIN0204_L3.6mm_D1.6mm_P2.54mm_Vertical -> Resistor_SMD:R_0805_2012Metric_Pad1.15x1.40mm_HandSolder
- moved R1 32.5 mm to (192.0, 76.7), turned to 180 degrees
- moved R3 25.2 mm to (192.0, 79.2), turned to 180 degrees
- moved J8 23.1 mm to (185.4, 106.7)
- moved J7 21.8 mm to (185.4, 101.6)
- moved J3 21.0 mm to (185.4, 63.5)
- moved J6 20.6 mm to (185.4, 96.5)
- moved J5 19.4 mm to (185.4, 91.4)
- moved J4 18.4 mm to (185.4, 78.7)
- moved R8 16.4 mm to (192.0, 108.7)
- moved R2 14.8 mm to (192.0, 81.8), turned to 180 degrees
- moved J2 12.4 mm to (185.4, 73.7), turned to 0 degrees
- moved R7 12.1 mm to (192.0, 102.6)
- moved R4 11.2 mm to (192.0, 84.3), turned to 180 degrees
- moved C1 11.0 mm to (187.9, 63.9), turned to 270 degrees
- moved Q4 10.8 mm to (192.0, 105.7), turned to 0 degrees
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Connections:
- net Net-(J5-Pad2) renamed /IRB_1
- net Net-(J6-Pad2) renamed /IRB_2
- net Net-(J7-Pad2) renamed /IRB_3
- net Net-(J8-Pad2) renamed /IRB_4
- J1 pad 2: /IR_OUT -> /5V
- J1 pad 3: /STATUS -> /IR_IN
- J1 pad 4: /IR_IN -> /5V
- J1 pad 5: /5V -> /STATUS
- J1 pad 6: /5V -> /GND
- J1 pad 7: /GND -> /IR_OUT
- J4 pad 3: Net-(J4-Pad3) -> /IR_IN
- J4 pad 5: /IR_IN -> Net-(J4-Pad5)
- Q1 pad 2: Net-(Q1-Pad2) -> /GND
- Q1 pad 3: /GND -> Net-(Q1-Pad3)
- Q2 pad 1: Net-(Q2-Pad1) -> Net-(Q1-Pad1)
- Q2 pad 2: Net-(Q1-Pad2) -> /GND
- Q2 pad 3: /GND -> Net-(Q2-Pad3)
- Q3 pad 1: Net-(Q3-Pad1) -> Net-(Q1-Pad1)
- Q3 pad 2: Net-(Q1-Pad2) -> /GND
- Q3 pad 3: /GND -> Net-(Q3-Pad3)
- Q4 pad 1: Net-(Q4-Pad1) -> Net-(Q1-Pad1)
- Q4 pad 2: Net-(Q1-Pad2) -> /GND
- Q4 pad 3: /GND -> Net-(Q4-Pad3)
- R3 pad 2: Net-(J4-Pad3) -> Net-(J4-Pad5)
- R4 pad 1: Net-(Q1-Pad2) -> Net-(Q1-Pad1)
- R5 pad 2: Net-(Q1-Pad1) -> Net-(Q1-Pad3)
- R6 pad 2: Net-(Q2-Pad1) -> Net-(Q2-Pad3)
- R7 pad 2: Net-(Q3-Pad1) -> Net-(Q3-Pad3)
- R8 pad 2: Net-(Q4-Pad1) -> Net-(Q4-Pad3)
Routing:
- net /12V: track 0.00 -> 44.7 mm
- net Net-(Q1-Pad1): track 0.00 -> 28.2 mm
- net /IR_IN: track 0.00 -> 19.9 mm
- net /3.3V: track 0.00 -> 17.9 mm
- net /IR_OUT: track 0.00 -> 16.0 mm
- net /5V: track 0.00 -> 12.4 mm, vias 0 -> 1
- net Net-(J4-Pad4): track 0.00 -> 12.0 mm
- net Net-(J4-Pad5): track 0.00 -> 12.0 mm
- net /STATUS: track 0.00 -> 9.18 mm
- net /IRB_1: track 0.00 -> 7.05 mm
- net /IRB_2: track 0.00 -> 6.63 mm
- net /IRB_3: track 0.00 -> 6.21 mm
- net /IRB_4: track 0.00 -> 5.79 mm
- net Net-(Q4-Pad3): track 0.00 -> 3.24 mm
- net Net-(Q1-Pad3): track 0.00 -> 3.24 mm
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- added copper zone on B.Cu, net /GND
- added copper zone on F.Cu, net /GND
Other:
- board size 28 x 48.3 mm -> 11.2 x 51.3 mm
- net class Default: clearance 0.2 -> 0.1524; trace_width 0.25 -> 0.1524; via_dia 0.8 -> 0.6858; via_drill 0.4 -> 0.3302
- net class IR added: clearance 0.1524, trace_width 0.4572, via_dia 0.6858, via_drill 0.3302
- net class Power added: clearance 0.1524, trace_width 0.4572, via_dia 0.6858, via_drill 0.3302
- net class Signal added: clearance 0.1524, trace_width 0.1778, via_dia 0.6858, via_drill 0.3302
- rule pad_to_mask_clearance: 0 -> 0.0508
- rule trace_clearance: 0.2 -> 0.1524
- rule trace_min: 0.2 -> 0.1524
- rule via_min_drill: 0.3 -> 0.254
- rule via_min_size: 0.4 -> 0.508

Commit message: New designs
Parts:
- removed R7, R8: 0, Resistor_SMD:R_0805_2012Metric_Pad1.15x1.40mm_HandSolder
- removed the REF** at (190.5, 111.8)
- added REF**: Support, Pin_Headers:Pin_Header_Straight_1x02_Pitch2.54mm, F.Cu at (147.3, 129.5)
- J4: value Front Panel 1 -> Front Panel
- R1: value 750 -> 10K
- R2: value 10K -> 100
- R3: value 750 -> 0
- R4: value 100 -> 0
- moved R4 53.1 mm to (148.2, 114.3), turned to 0 degrees
- moved R5 53.1 mm to (148.2, 120.4)
- moved R6 53.0 mm to (148.2, 126.4)
- moved R3 52.5 mm to (148.2, 108.2), turned to 0 degrees
- moved R1 49.6 mm to (148.2, 99.9), turned to 0 degrees
- moved R2 48.3 mm to (148.2, 102.2)
- moved C1 47.8 mm to (148.9, 91.5), turned to 0 degrees
- moved Q1 47.3 mm to (148.2, 105.2)
- moved Q2 47.3 mm to (148.2, 111.3)
- moved Q3 47.3 mm to (148.2, 117.3)
- moved Q4 47.3 mm to (148.2, 123.4)
- moved J1 46.7 mm to (147.3, 81.3)
- moved J2 45.3 mm to (143.8, 91.4)
- moved J3 45.3 mm to (143.8, 81.3)
- moved J4 45.3 mm to (143.8, 96.5)
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Connections:
- J4 pad 4: Net-(J4-Pad4) -> /STATUS
- J4 pad 5: Net-(J4-Pad5) -> /IR_OUT
- R1 pad 1: /STATUS -> /IR_OUT
- R1 pad 2: Net-(J4-Pad4) -> /GND
- R2 pad 1: /IR_OUT -> Net-(Q1-Pad1)
- R2 pad 2: /GND -> /IR_OUT
- R3 pad 1: /IR_OUT -> /IRB_1
- R3 pad 2: Net-(J4-Pad5) -> Net-(Q1-Pad3)
- R4 pad 1: Net-(Q1-Pad1) -> /IRB_2
- R4 pad 2: /IR_OUT -> Net-(Q2-Pad3)
- R5 pad 1: /IRB_1 -> /IRB_3
- R5 pad 2: Net-(Q1-Pad3) -> Net-(Q3-Pad3)
- R6 pad 1: /IRB_2 -> /IRB_4
- R6 pad 2: Net-(Q2-Pad3) -> Net-(Q4-Pad3)
Routing:
- net Net-(J4-Pad4): track 12.0 -> 0.00 mm
- net Net-(J4-Pad5): track 12.0 -> 0.00 mm
- net /STATUS: track 9.18 -> 19.3 mm
- net /5V: track 12.4 -> 18.2 mm, vias 1 -> 0
- net /IR_OUT: track 16.0 -> 20.1 mm
- net /GND: track 2.97 -> 0.00 mm, vias 8 -> 15
- net /IRB_3: track 6.21 -> 4.05 mm
- net /IRB_2: track 6.63 -> 4.47 mm
- net /IRB_4: track 5.79 -> 3.66 mm
- net Net-(Q1-Pad1): track 28.2 -> 26.6 mm
- net /IRB_1: track 7.05 -> 5.49 mm
- net /3.3V: track 17.9 -> 16.7 mm
- net /12V: track 44.7 -> 43.9 mm
- net /IR_IN: track 19.9 -> 19.3 mm
Other:
- board size 11.2 x 51.3 mm -> 9.1 x 50.8 mm
- board text added: "+"
- board text added: "1"
- board text added: "IRBlaster v1"
