File: PCBs/Interface/Interface.sch (KiCad schematic (older format))
At the start: 43 parts, among them J1 MCU, J2 VLED, SW11 SW_Push, SW13 SW_Push, SW14 SW_Push, SW15 SW_Push, SW16 SW_Push, SW21 SW_Push, SW22 SW_Push, SW23 SW_Push, SW24 SW_Push, SW25 SW_Push, SW26 SW_Push, SW31 SW_Push, SW32 SW_Push, SW35 SW_Push, SW36 SW_Push, SW41 SW_Push, SW42 SW_Push, SW43 SW_Push, SW44 SW_Push, SW45 SW_Push, SW51 SW_Push, SW52 SW_Push, SW53 SW_Push, SW54 SW_Push, SW55 SW_Push, SW56 SW_Push, SW61 SW_Push, SW62 SW_Push, SW63 SW_Push, SW64 SW_Push, SW66 SW_Push

Commit message: Hopefullly final design before manufacture
Parts:
- removed SW22: SW_Push, my-switches:SMD_MultiSwitch, symbol Switch:SW_Push
- J1: footprint Pin_Headers:Pin_Header_Angled_1x13_Pitch2.54mm -> my-smd:SMD_Right_Socket_Strip_Angled_1x13_Pitch2.54mm
- J2: footprint Pin_Headers:Pin_Header_Angled_1x02_Pitch2.54mm -> my-smd:SMD_Right_Socket_Strip_Angled_1x02_Pitch2.54mm
- SW11, SW13, SW14, SW15, SW16, SW21, SW23, SW24, SW25, SW26, SW31, SW32, SW35, SW36, SW41, SW42, SW43, SW44, SW45, SW51, SW52, SW53, SW54, SW55, SW56, SW61, SW62, SW63, SW64, SW66: footprint my-switches:SMD_MultiSwitch -> my-switches:SMD_Tactile_Switch
Connections:
- net COL1: now also J1.13 (Pin_13); no longer J1.8 (Pin_8)
- net COL2: now also J1.11 (Pin_11); no longer J1.9 (Pin_9)
- net COL3: now also J1.9 (Pin_9); no longer J1.10 (Pin_10)
- net COL4: now also J1.12 (Pin_12); no longer J1.11 (Pin_11)
- net COL5: now also J1.10 (Pin_10); no longer J1.12 (Pin_12)
- net COL6: now also J1.8 (Pin_8); no longer J1.13 (Pin_13)

Commit message: Changed decoupling cap values
Parts:
- C1, C2, C3, C4, C5: value 1uF -> 0.1uF
Changed lines of the file:
@@
 P 2900 2200
 F 0 "C1" H 3015 2246 50  0000 L CNN
-F 1 "1uF" H 3015 2155 50  0000 L CNN
+F 1 "0.1uF" H 3015 2155 50  0000 L CNN
 F 2 "Capacitors_SMD:C_0805_HandSoldering" H 2938 2050 50  0001 C CNN
 F 3 "~" H 2900 2200 50  0001 C CNN
@@
 P 4000 2200
 F 0 "C2" H 4115 2246 50  0000 L CNN
-F 1 "1uF" H 4115 2155 50  0000 L CNN
+F 1 "0.1uF" H 4115 2155 50  0000 L CNN
 F 2 "Capacitors_SMD:C_0805_HandSoldering" H 4038 2050 50  0001 C CNN
 F 3 "~" H 4000 2200 50  0001 C CNN
@@
 P 6200 2200
 F 0 "C4" H 6315 2246 50  0000 L CNN
-F 1 "1uF" H 6315 2155 50  0000 L CNN
+F 1 "0.1uF" H 6315 2155 50  0000 L CNN
 F 2 "Capacitors_SMD:C_0805_HandSoldering" H 6238 2050 50  0001 C CNN
 F 3 "~" H 6200 2200 50  0001 C CNN
@@
 P 5100 2200
 F 0 "C3" H 5215 2246 50  0000 L CNN
-F 1 "1uF" H 5215 2155 50  0000 L CNN
+F 1 "0.1uF" H 5215 2155 50  0000 L CNN
 F 2 "Capacitors_SMD:C_0805_HandSoldering" H 5138 2050 50  0001 C CNN
 F 3 "~" H 5100 2200 50  0001 C CNN
@@
 P 7300 2200
 F 0 "C5" H 7415 2246 50  0000 L CNN
-F 1 "1uF" H 7415 2155 50  0000 L CNN
+F 1 "0.1uF" H 7415 2155 50  0000 L CNN
 F 2 "Capacitors_SMD:C_0805_HandSoldering" H 7338 2050 50  0001 C CNN
 F 3 "~" H 7300 2200 50  0001 C CNN
